Commit message: Add 29dof dataset conversion utils

File: assets/g1/g1_29dof_custom.urdf (robot description, URDF)
Before this commit: robot g1_29dof_rev_1_0, 39 links, 38 joints
Links:
- added link head_mocap
Joints:
- added joint head_mocap_joint: type fixed, parent torso_link, child head_mocap, origin xyz=0 0 0.4 rpy=0 0 0

Commit message: Refactor 29‑DOF G1 pipeline and configs; remove 23‑DOF fallbacks

File: assets/g1/g1_29dof_custom.urdf (robot description, URDF)
Before this commit: robot g1_29dof_rev_1_0, 40 links, 39 joints
Links:
- removed link d435_link
- removed link imu_in_pelvis
- removed link logo_link
- removed link mid360_link
- added link left_toe_link
- added link right_toe_link
Joints:
- removed joint d435_joint
- removed joint imu_in_pelvis_joint
- removed joint logo_joint
- removed joint mid360_joint
- added joint left_toe_joint: type fixed, parent left_ankle_roll_link, child left_toe_link, origin xyz=0.12 0.0 -0.039 rpy=0 0 0
- added joint right_toe_joint: type fixed, parent right_ankle_roll_link, child right_toe_link, origin xyz=0.12 0.0 -0.039 rpy=0 0 0
